File: PCB/LP_Monitor/lpmon.sch (EAGLE design)
At the start: 9 parts, among them U1 ATMEGA328P-PU

Commit message: started pcb
Parts:
- added UART_HEAD: (no value), pinhead:PINHD-1X3
Connections:
- net CH_EN: now also U1.PD3
- net GND: now also UART_HEAD.1
- net W_RX: now also U1.PD1, UART_HEAD.3
- net W_TX: now also U1.PD0, UART_HEAD.2
Changed lines of the file:
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@@
 <part name="X_4" library="ngspice-simulation" library_urn="urn:adsk.eagle:library:527439" deviceset="GND" device=""/>
 <part name="WIFI" library="con-lstb" library_urn="urn:adsk.eagle:library:162" deviceset="MA04-2" device="" package3d_urn="urn:adsk.eagle:package:8368/1"/>
+<part name="UART_HEAD" library="pinhead" library_urn="urn:adsk.eagle:library:325" deviceset="PINHD-1X3" device="" package3d_urn="urn:adsk.eagle:package:22458/2"/>
 </parts>
 <sheets>
@@
 <attribute name="VALUE" x="-29.21" y="43.18" size="1.778" layer="96"/>
 <attribute name="NAME" x="-29.21" y="59.182" size="1.778" layer="95"/>
+</instance>
+<instance part="UART_HEAD" gate="A" x="-27.94" y="78.74" smashed="yes" rot="R180">
+<attribute name="NAME" x="-21.59" y="73.025" size="1.778" layer="95" rot="R180"/>
+<attribute name="VALUE" x="-21.59" y="86.36" size="1.778" layer="96" rot="R180"/>
 </instance>
 </instances>
@@
 <label x="-12.7" y="55.88" size="1.778" layer="95"/>
 </segment>
+<segment>
+<pinref part="UART_HEAD" gate="A" pin="1"/>
+<wire x1="-25.4" y1="76.2" x2="-17.78" y2="76.2" width="0.1524" layer="91"/>
+<label x="-17.78" y="76.2" size="1.778" layer="95"/>
+</segment>
 </net>
 <net name="3V3" class="0">
@@
 <segment>
 <pinref part="U1" gate="A" pin="PC6"/>
-<wire x1="78.74" y1="40.64" x2="91.44" y2="40.64" width="0.1524" layer="91"/>
-<label x="91.44" y="40.64" size="1.27" layer="95" xref="yes"/>
+<wire x1="78.74" y1="40.64" x2="86.36" y2="40.64" width="0.1524" layer="91"/>
+<label x="86.36" y="40.64" size="1.27" layer="95" xref="yes"/>
 </segment>
 <segment>
@@
 <label x="-12.7" y="48.26" size="1.778" layer="95" xref="yes"/>
 </segment>
+<segment>
+<pinref part="U1" gate="A" pin="PD1"/>
+<wire x1="78.74" y1="76.2" x2="83.82" y2="76.2" width="0.1524" layer="91"/>
+<label x="83.82" y="76.2" size="1.016" layer="95" xref="yes"/>
+</segment>
+<segment>
+<pinref part="UART_HEAD" gate="A" pin="3"/>
+<wire x1="-25.4" y1="81.28" x2="-17.78" y2="81.28" width="0.1524" layer="91"/>
+<label x="-17.78" y="81.28" size="1.778" layer="95"/>
+</segment>
 </net>
 <net name="CH_EN" class="0">
@@
 <label x="-40.64" y="53.34" size="1.778" layer="95"/>
 </segment>
+<segment>
+<pinref part="U1" gate="A" pin="PD3"/>
+<wire x1="78.74" y1="71.12" x2="86.36" y2="71.12" width="0.1524" layer="91"/>
+<label x="86.36" y="71.12" size="1.778" layer="95"/>
+</segment>
 </net>
 <net name="W_TX" class="0">
@@
 <label x="-43.18" y="55.88" size="1.778" layer="95" rot="R180" xref="yes"/>
 </segment>
-</net>
+<segment>
+<pinref part="U1" gate="A" pin="PD0"/>
+<wire x1="78.74" y1="78.74" x2="83.82" y2="78.74" width="0.1524" layer="91"/>
+<label x="83.82" y="78.74" size="1.016" layer="95" xref="yes"/>
+</segment>
+<segment>
+<pinref part="UART_HEAD" gate="A" pin="2"/>
+<wire x1="-25.4" y1="78.74" x2="-17.78" y2="78.74" width="0.1524" layer="91"/>
+<label x="-17.78" y="78.74" size="1.778" layer="95"/>
+</segment>
+</net>
